File: FN32ROV-XEBook-LED-KiCad.kicad_sch (KiCad schematic)
At the start: 4 parts, among them J1 LED_JST

Commit message: Switch J1 back to through-hole, grow board to 40x14mm, add logo, export fab files
Assembling both sides (SMD LEDs on front + SMD JST on back) was too costly for
JLCPCB assembly, so J1 reverts to through-hole and gets hand-soldered instead.
That meant reworking the board height and LED/connector Y-offsets so the
through-hole housing does not physically collide with the case light-pipe
housings (the earlier SMD-based clearance math did not carry over, since THT
housings are much deeper than the SMD footprint was).

Board is now 40x14mm: LEDs at y=3mm, mounting holes + J1 housing edge on the
y=7mm row, J1 pad row at y=9.2mm. Logo centered exactly on the back silkscreen.
LCSC part numbers recorded on each part in the schematic (D1=C471422,
D2=C30584803, D3=C28310436, J1=C265289). Fab export regenerated to match:
Gerbers, drill files, BOM/CPL (including a JLCPCB-Assembly-specific set that
excludes J1, since it is hand-soldered, not SMT-placed).

Co-Authored-By: Claude Sonnet 5 <noreply@anthropic.com>
Claude-Session: https://claude.ai/code/session_011E5FphyrLWBpYvbXpCPZfr
Parts:
- D1: LCSC (none) -> C471422
- D2: LCSC (none) -> C30584803
- D3: LCSC (none) -> C28310436
- J1: footprint Connector_JST:JST_PH_B4B-PH-SM4-TB_1x04-1MP_P2.00mm_Vertical -> Connector_JST:JST_PH_B4B-PH-K_1x04_P2.00mm_Vertical; LCSC (none) -> C265289
Changed lines of the file:
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@@
 			)
 		)
-		(property "Footprint" "Connector_JST:JST_PH_B4B-PH-SM4-TB_1x04-1MP_P2.00mm_Vertical"
-			(at 152.4 55.88 0)
-			(effects
-				(font
-					(size 1.27 1.27)
-				)
-				(hide yes)
-			)
-		)
-		(property "Datasheet" "~"
-			(at 152.4 55.88 0)
-			(effects
-				(font
-					(size 1.27 1.27)
-				)
-				(hide yes)
-			)
-		)
-		(property "Description" "Mates via 4-pin JST PH pigtail to J_LED1 on the FN32ROV-XEBook main board. SMD, mounted on the back (B.Cu) of this board -- surface mount so no through-hole barrel pokes through to the light-pipe side."
+		(property "Footprint" "Connector_JST:JST_PH_B4B-PH-K_1x04_P2.00mm_Vertical"
+			(at 152.4 55.88 0)
+			(effects
+				(font
+					(size 1.27 1.27)
+				)
+				(hide yes)
+			)
+		)
+		(property "Datasheet" "~"
+			(at 152.4 55.88 0)
+			(effects
+				(font
+					(size 1.27 1.27)
+				)
+				(hide yes)
+			)
+		)
+		(property "Description" "Mates via 4-pin JST PH pigtail to J_LED1 on the FN32ROV-XEBook main board. Through-hole, hand-soldered, mounted on the back of this board -- kept far enough (in Y) from the LED row that its plated-through pads do not land near the light-pipe contact points."
+			(at 152.4 55.88 0)
+			(effects
+				(font
+					(size 1.27 1.27)
+				)
+				(hide yes)
+			)
+		)
+		(property "LCSC" "C265289"
 			(at 152.4 55.88 0)
 			(effects
@@
 			)
 		)
-		(property "Description" "OSRAM LB QH9G-N1OO-35-1, blue. Carried over from original FN32ROV-1.7.1 BOM."
+		(property "Description" "YONGYUTAI YLED0402B, blue 460nm, Vf 2.6-3.1V."
+			(at 85.09 59.69 0)
+			(effects
+				(font
+					(size 1.27 1.27)
+				)
+				(hide yes)
+			)
+		)
+		(property "LCSC" "C30584803"
 			(at 85.09 59.69 0)
 			(effects
@@
 			)
 		)
-		(property "Description" "Rohm SML-P12DTT86R, orange. Carried over from original FN32ROV-1.7.1 BOM."
+		(property "Description" "YONGYUTAI YLED0402O, orange 611nm, Vf 1.8-2.3V."
+			(at 85.09 44.45 0)
+			(effects
+				(font
+					(size 1.27 1.27)
+				)
+				(hide yes)
+			)
+		)
+		(property "LCSC" "C28310436"
 			(at 85.09 44.45 0)
 			(effects
@@
 			)
 		)
-		(property "Description" "Rohm SML-P12PTT86R, green 560nm, Vf approx 2.2V typ. Replaces original SunLED white LED for this board (see main board R13)."
-			(at 85.09 74.93 0)
-			(effects
+		(property "Description" "Everlight 16-213/G6C-AK2L2VY/3T, yellow-green 575nm, Vf 1.7-2.2V. Replaces original SunLED white LED for this board (see main board R13)."
+			(at 85.09 74.93 0)
+			(effects
+				(font
+					(size 1.27 1.27)
+				)
+				(hide yes)
+			)
+		)
+		(property "LCSC" "C471422"
+			(at 85.09 74.93 0)
+			(effects
